Commit message: feat : add launch file for rviz visualization

File: urdf/quad.urdf (robot description, URDF)
Before this commit: robot quad_f450_camera, 8 links, 7 joints
Links:
- link /camera_quad_f450_link: geometry collision box size=0.023813 0.027686 0.092682; visual mesh filename=package://quadrotor_sim/meshes/cam_link.STL
- link base_link_inertia: geometry collision box size=0.3585 0.3585 0.22; visual mesh filename=package://quadrotor_sim/meshes/base_link.STL scale=1 1 1
- link rotor_0: geometry collision cylinder length=0.005 radius=0.065; visual mesh filename=package://quadrotor_sim/meshes/propeller_1.STL scale=1 1 1
- link rotor_1: geometry collision cylinder length=0.005 radius=0.065; visual mesh filename=package://quadrotor_sim/meshes/propeller_1.STL scale=1 1 1
- link rotor_2: geometry collision cylinder length=0.005 radius=0.065; visual mesh filename=package://quadrotor_sim/meshes/propeller_0.STL scale=1 1 1
- link rotor_3: geometry collision cylinder length=0.005 radius=0.065; visual mesh filename=package://quadrotor_sim/meshes/propeller_0.STL scale=1 1 1

File: urdf/quad.xacro (robot description, xacro)
@@ -66,5 +66,5 @@
   </xacro:property>
   <!-- Included URDF Files -->
-  <xacro:include filename="$(arg quad_f450_camera_dir)/urdf/multirotor_base.xacro" />
+  <xacro:include filename="$(find quadrotor_sim)/urdf/multirotor_base.xacro" />
   <!-- Instantiate multirotor_base_macro once -->
   <xacro:multirotor_base_macro

File: urdf/quad_base.xacro (robot description, xacro)
@@ -1,8 +1,8 @@
 <?xml version="1.0"?>
-<robot name="quad_f450_camera" xmlns:xacro="http://ros.org/wiki/xacro">
+<robot name="quadrotor_f450" xmlns:xacro="http://ros.org/wiki/xacro">
   <!-- Properties that can be assigned at build time as arguments.
   Is there a reason not to make all properties arguments?
   -->
-  <xacro:arg name='name' default='quad_f450_camera' />
+  <xacro:arg name='name' default='quadrotor_f450' />
   <xacro:arg name='mavlink_addr' default='INADDR_ANY' />
   <xacro:arg name='mavlink_udp_port' default='14560' />
@@ -17,5 +17,5 @@
   <xacro:arg name='hil_mode' default='false' />
   <xacro:arg name='hil_state_level' default='false' />
-  <xacro:arg name='send_vision_estimation' default='true' />
+  <xacro:arg name='send_vision_estimation' default='false' />
   <xacro:arg name='send_odometry' default='false' />
   <xacro:arg name='enable_lockstep' default='true' />
@@ -23,14 +23,13 @@
   <xacro:arg name='vehicle_is_tailsitter' default='false' />
   <xacro:arg name='visual_material' default='DarkGrey' />
-  <xacro:arg name='enable_mavlink_interface' default='true' />
+  <xacro:arg name='enable_mavlink_interface' default='false' />
   <xacro:arg name='enable_wind' default='false' />
-  <!-- The following causes segfault with multiple vehicles if defaults to true!!! -->
   <xacro:arg name='enable_ground_truth' default='false' />
   <xacro:arg name='enable_logging' default='false' />
-  <xacro:arg name='log_file' default='quad_f450_camera' />
+  <xacro:arg name='log_file' default='quadrotor_f450' />
   <!-- macros for gazebo plugins, sensors -->
-  <xacro:include filename="$(arg quad_f450_camera_dir)/urdf/component_snippets.xacro" />
+  <xacro:include filename="$(find quadrotor_sim)/urdf/component_snippets.xacro" />
   <!-- Instantiate iris "mechanics" -->
-  <xacro:include filename="$(arg quad_f450_camera_dir)/urdf/quad.xacro" />
+  <xacro:include filename="$(find quadrotor_sim)/urdf/quad.xacro" />
   <xacro:if value="$(arg enable_wind)">
     <xacro:wind_plugin_macro
