Commit message: fix : minor changes

File: urdf/component_snippets.xacro (robot description, xacro)
@@ -50,5 +50,7 @@
             <mesh filename="package://quadrotor_sim/meshes/cam_link.STL" />
           </geometry>
-          <material name="red" />
+          <material name="red">
+            <color rgba="0.8 0.0 0.0 1.0"/>
+          </material>
         </visual>
       </xacro:if>

File: urdf/quad.xacro (robot description, xacro)
@@ -1,4 +1,4 @@
 <?xml version="1.0"?>
-<robot name="quad_f450_camera" xmlns:xacro="http://ros.org/wiki/xacro">
+<robot name="quadrotor_f450" xmlns:xacro="http://ros.org/wiki/xacro">
   <!-- Properties -->
   <xacro:property name="namespace" value="" />

Commit message: fix : temp solution to import meshes

File: urdf/component_snippets.xacro (robot description, xacro)
@@ -48,5 +48,5 @@
           <origin xyz="0 0 0" rpy="0 0 0" />
           <geometry>
-            <mesh filename="package://quadrotor_sim/meshes/cam_link.STL" />
+            <mesh filename="/home/shaswatgarg/quadROS/src/quadrotor_sim/meshes/cam_link.STL" />
           </geometry>
           <material name="red">

File: urdf/multirotor_base.xacro (robot description, xacro)
@@ -35,5 +35,5 @@
         <origin xyz="0 0 0" rpy="0 0 0" />
         <geometry>
-          <mesh filename="package://quadrotor_sim/meshes/${mesh_file}"
+          <mesh filename="/home/shaswatgarg/quadROS/src/quadrotor_sim/meshes/${mesh_file}"
             scale="${mesh_scale}" />
           <!-- <box size="${body_width} ${body_width} ${body_height}"/> --> <!-- [m] [m] [m] -->
@@ -95,5 +95,5 @@
           <!-- <cylinder length="0.005" radius="${radius_rotor}"/> --> <!-- [m] -->
           <!-- <mesh filename="package://rotors_description/meshes/propeller_${direction}.dae" -->
-          <mesh filename="package://quadrotor_sim/meshes/${mesh}.STL"
+          <mesh filename="/home/shaswatgarg/quadROS/src/quadrotor_sim/meshes/${mesh}.STL"
             scale="${mesh_scale}" />
           <!-- <box size="${2*radius_rotor} 0.01 0.005"/> -->

File: urdf/quad_base.xacro (robot description, xacro)
@@ -45,11 +45,11 @@
   </xacro:if>
   <!-- Instantiate gps plugin. -->
-  <xacro:gps_plugin_macro
+  <!-- <xacro:gps_plugin_macro
     namespace="${namespace}"
     gps_noise="true"
     >
-  </xacro:gps_plugin_macro>
+  </xacro:gps_plugin_macro> -->
   <!-- Instantiate magnetometer plugin. -->
-  <xacro:magnetometer_plugin_macro
+  <!-- <xacro:magnetometer_plugin_macro
     namespace="${namespace}"
     pub_rate="50"
@@ -59,14 +59,14 @@
     mag_topic="/mag"
     >
-  </xacro:magnetometer_plugin_macro>
+  </xacro:magnetometer_plugin_macro> -->
   <!-- Instantiate barometer plugin. -->
-  <xacro:barometer_plugin_macro
+  <!-- <xacro:barometer_plugin_macro
     namespace="${namespace}"
     pub_rate="50"
     baro_topic="/baro"
     >
-  </xacro:barometer_plugin_macro>
+  </xacro:barometer_plugin_macro> -->
   <!-- Instantiate GroundTruth plugin. -->
-  <xacro:ground_truth_plugin_macro
+  <!-- <xacro:ground_truth_plugin_macro
     base="base_link"
     pub_rate="30"
@@ -74,4 +74,5 @@
     >
   </xacro:ground_truth_plugin_macro>
+ -->
   <xacro:if value="$(arg enable_mavlink_interface)">
   <!-- Instantiate mavlink telemetry interface. -->
@@ -102,5 +103,5 @@
   </xacro:mavlink_interface_macro>
   </xacro:if>
-  <xacro:camera_macro
+  <!-- <xacro:camera_macro
     namespace="${namespace}"
     parent_link="base_link"
@@ -117,9 +118,9 @@
     enable_visual="1"
   >
-  <box size="0.01 0.01 0.01" />   <!-- 0.05 -->
-  <origin xyz="0 0 -0.013633" rpy="1.5708 1.5708 0"/>  <!-- 0.07 -->
-  </xacro:camera_macro>
+  <box size="0.01 0.01 0.01" />
+  <origin xyz="0 0 -0.013633" rpy="1.5708 1.5708 0"/>
+  </xacro:camera_macro> -->
   <!-- Mount an ADIS16448 IMU. -->
-  <xacro:imu_plugin_macro
+  <!-- <xacro:imu_plugin_macro
     namespace="${namespace}"
     imu_suffix=""
@@ -138,5 +139,5 @@
     <inertia ixx="0.00001" ixy="0.0" ixz="0.0" iyy="0.00001" iyz="0.0" izz="0.00001" />
     <origin xyz="0 0 0" rpy="0 0 0" />
-  </xacro:imu_plugin_macro>
+  </xacro:imu_plugin_macro> -->
   <xacro:if value="$(arg enable_ground_truth)">
     <!-- Mount an IMU providing ground truth. -->
